Commit message: send the camera transform automatically using 'robot_state_publisher'

File: a1_description/xacro/robot_cut.xacro (robot description, xacro)
@@ -109,4 +109,29 @@
         </collision>
     </link>
+    <joint name="camera_joint" type="fixed">
+        <parent link="trunk"/>
+        <child link="range-finder"/>
+        <origin rpy="0 0.2618 0" xyz="0.2633438 0 0.0301362"/>
+    </joint>
+    <link name="range-finder">
+        <inertial>
+            <mass value="0.001"/>
+            <origin rpy="0 0 0" xyz="0 0 0"/>
+            <inertia ixx="0.0001" ixy="0" ixz="0" iyy="0.0001" iyz="0" izz="0.0001"/>
+        </inertial>
+        <visual>
+            <origin rpy="0 0 0" xyz="0 0 0"/>
+            <geometry>
+                <box size="0.001 0.001 0.001"/>
+            </geometry>
+            <material name="red"/>
+        </visual>
+        <collision>
+            <origin rpy="0 0 0" xyz="0 0 0"/>
+            <geometry>
+                <box size=".001 .001 .001"/>
+            </geometry>
+        </collision>
+    </link>
     <xacro:leg name="FR" mirror="-1" mirror_dae="False" front_hind="1" front_hind_dae="True">
         <origin rpy="0 0 0" xyz="${leg_offset_x} ${-leg_offset_y} 0"/>
